File: kicad/power-distribution-board.kicad_sch (KiCad schematic)
At the start: 15 parts, among them J1 Banana Socket PCBMount, J2 Banana Socket PCBMount, J3 Banana Socket PCBMount, J4 Conn_02x08_Odd_Even, J5 Conn_02x05_Odd_Even, J6 4U_Power, J7 Conn_01x03, SW1 SW_DPDT_x2

Commit message: Adding pcb layout
Parts:
- added D3, D4: 1N4001, Rumblesan_Standard_Parts:D_DO-41_SOD81_P10.16mm_Horizontal, symbol Device:D
- added H1, H2, H3, H4: MountingHole_Pad, MountingHole:MountingHole_3.2mm_M3_DIN965_Pad, symbol Mechanical:MountingHole_Pad
- added J10, J8, J9: Banana Socket PCBMount, Rumblesan_Audio_Connectors:Deltron_571_PCB_BananaJack, symbol Rumblesan_Banana_Jacks:Banana_Socket_PCBMount
- added J11: Conn_01x04, Connector_Molex:Molex_KK-396_5273-04A_1x04_P3.96mm_Vertical, symbol Connector_Generic:Conn_01x04
- D1, D2: footprint (none) -> LED_THT:LED_D5.0mm
- J6: footprint 4U_Power:4u_Power_Molex_KK-254_P2.54mm -> Rumblesan_4U_Power:4u_Power_Molex_KK-254_22-27-2041_1x04_P2.54mm_Vertical
- J7: footprint (none) -> Connector_Molex:Molex_KK-254_AE-6410-03A_1x03_P2.54mm_Vertical
- SW1: footprint (none) -> Rumblesan_Standard_Parts:SW_DPDT_DailyWell_MiniToggle
- TP1, TP2, TP3: footprint (none) -> Rumblesan_Standard_Parts:TestPoint_Loop_D2.50mm_Drill1.0mm_LowProfile
Connections:
- net +12V: now also J11.1 (Pin_1), J8.1
- net -12V: now also J11.4 (Pin_4), J9.1
- net GND: now also D3.2 (A), D4.1 (K), H1.1, H2.1, H3.1, H4.1, J10.1, J11.2 (Pin_2), J11.3 (Pin_3)
- net at J2.1, SW1.4 (A): now also D4.2 (A)
- net at J1.1, SW1.1 (A): now also D3.1 (K)
Other:
- moved on the sheet: D1, J1, J2, R1, SW1A, TP2, TP3

Commit message: Tweaking layout and adding silkscreen text
Parts:
- TP1, TP2, TP3: now left out of the parts list
Other:
- company: (none) -> Helical Sounds
- title: (none) -> Power Distribution Helper
Changed lines of the file:
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@@
 	(paper "A4")
 	(title_block
+		(title "Power Distribution Helper")
+		(date "2025-02-13")
+		(rev "r01")
+		(company "Helical Sounds")
 		(comment 2 "creativecommons.org/licenses/by/4.0/")
 		(comment 3 "License: CC BY 4.0")
@@
 		(unit 1)
 		(exclude_from_sim no)
-		(in_bom yes)
+		(in_bom no)
 		(on_board yes)
 		(dnp no)
@@
 		(unit 1)
 		(exclude_from_sim no)
-		(in_bom yes)
+		(in_bom no)
 		(on_board yes)
 		(dnp no)
@@
 		(unit 1)
 		(exclude_from_sim no)
-		(in_bom yes)
+		(in_bom no)
 		(on_board yes)
 		(dnp no)
